File: hardware/Glassboard.kicad_sch (KiCad schematic)
At the start: 18 parts, among them J1 Conn_01x03, U1 NT3H2111W0FTTJ, U2 ATtiny202-SS

Commit message: fixed schematic names
Parts:
- renumbered C_VOUT1 to C2, C_RESET1 to C3, D_LED1 to D1, D_LED2 to D2, D_LED3 to D3
Changed lines of the file:
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@@
 		(on_board yes)
 		(dnp no)
-		(property "Reference" "D_LED1"
+		(property "Reference" "D1"
 			(at 232.7275 85.09 0)
 			(effects
@@
 			(project "Glassboard"
 				(path "/1451c52f-1bb9-4a48-ad08-fcf3fedff30a"
-					(reference "D_LED1")
+					(reference "D1")
 					(unit 1)
 				)
@@
 		(dnp no)
 		(fields_autoplaced yes)
-		(property "Reference" "C_RESET1"
+		(property "Reference" "C3"
 			(at 204.47 88.8999 0)
 			(effects
@@
 			(project ""
 				(path "/1451c52f-1bb9-4a48-ad08-fcf3fedff30a"
-					(reference "C_RESET1")
+					(reference "C3")
 					(unit 1)
 				)
@@
 		(on_board yes)
 		(dnp no)
-		(property "Reference" "D_LED3"
+		(property "Reference" "D3"
 			(at 249.2375 115.57 0)
 			(effects
@@
 			(project ""
 				(path "/1451c52f-1bb9-4a48-ad08-fcf3fedff30a"
-					(reference "D_LED3")
+					(reference "D3")
 					(unit 1)
 				)
@@
 		(on_board yes)
 		(dnp no)
-		(property "Reference" "D_LED2"
+		(property "Reference" "D2"
 			(at 255.5875 101.6 0)
 			(effects
@@
 			(project "Glassboard"
 				(path "/1451c52f-1bb9-4a48-ad08-fcf3fedff30a"
-					(reference "D_LED2")
+					(reference "D2")
 					(unit 1)
 				)
@@
 		(dnp no)
 		(fields_autoplaced yes)
-		(property "Reference" "C_VOUT1"
+		(property "Reference" "C2"
 			(at 134.62 105.4099 0)
 			(effects
@@
 			(project ""
 				(path "/1451c52f-1bb9-4a48-ad08-fcf3fedff30a"
-					(reference "C_VOUT1")
-					(unit 1)
-				)
+					(reference "C2")
+					(unit 1)
+				)
